Commit message: Naman | Figures out the navigation

File: src/ugv_main/ugv_description/urdf/ugv_rover.urdf (robot description, URDF)
Before this commit: robot ugv_rover, 13 links, 12 joints
Links:
- added link overhead_camera_link, mass 0.005; collision box size=0.03 0.025 0.02; visual box size=0.03 0.025 0.02
Joints:
- added joint pt_camera_to_overhead_camera_joint: type fixed, parent pt_camera_link, child overhead_camera_link, origin xyz=0 0 0.035 rpy=0 0 0, axis 0 0 0
